File: STM32H7A3RGT6_Devboard.kicad_sch (KiCad schematic)
At the start: 11 parts, among them U1 STM32H7A3RGT6

Commit message: First full draft
Parts:
- added C11, C12: 1uF, Capacitor_SMD:C_0402_1005Metric_Pad0.74x0.62mm_HandSolder, symbol Device:C
- added C13, C14: 8pF, Capacitor_SMD:C_0402_1005Metric_Pad0.74x0.62mm_HandSolder, symbol Device:C
- added C15: 1uF, Capacitor_SMD:C_0603_1608Metric_Pad1.08x0.95mm_HandSolder, symbol Device:C
- added D1: DF2B7AE, Diode_SMD:D_SOD-523, symbol Device:D
- added D2, D3: LED, LED_SMD:LED_0603_1608Metric, symbol Device:LED
- added J1: USB_C_Receptacle_USB2.0_14P, USBC:USB_C_Receptacle_Molex_217179-0001, symbol Connector:USB_C_Receptacle_USB2.0_14P
- added J2: Conn_01x04_Socket, Connector_PinHeader_2.54mm:PinHeader_1x04_P2.54mm_Vertical, symbol Connector:Conn_01x04_Socket
- added J3, J4: Conn_01x25_PinHeader, Connector_PinHeader_2.54mm:PinHeader_1x25_P2.54mm_Vertical, symbol Connector:Conn_01x25_Socket
- added R1, R2, R4, R5: 5k1, Resistor_SMD:R_0603_1608Metric, symbol Device:R
- added R3, R6: 1k, Resistor_SMD:R_0603_1608Metric_Pad0.98x0.95mm_HandSolder, symbol Device:R
- added SW1: RESET, Button_Switch_SMD:SW_Push_1P1T-SH_NO_CK_KMR2xxG, symbol Switch:SW_Push
- added SW2: BOOT, Button_Switch_SMD:SW_Push_1P1T-SH_NO_CK_KMR2xxG, symbol Switch:SW_Push
- added U2: AP2127N-3.3TRG1, Package_TO_SOT_SMD:SOT-23, symbol Regulator_Linear:AP2127N-3.3
- added U3: USBLC6-2SC6, Package_TO_SOT_SMD:SOT-23-6, symbol Power_Protection:USBLC6-2SC6
- added Y1: 12MHz, Crystal:Crystal_SMD_2016-4Pin_2.0x1.6mm, symbol Device:Crystal_GND24
- C1: footprint Package_QFP:LQFP-64_10x10mm_P0.5mm -> Capacitor_SMD:C_0402_1005Metric_Pad0.74x0.62mm_HandSolder
- C10, C2, C3, C4, C5, C6, C7, C9: footprint (none) -> Capacitor_SMD:C_0402_1005Metric_Pad0.74x0.62mm_HandSolder
- C8: footprint (none) -> Capacitor_SMD:C_0603_1608Metric
Connections:
- net +3V3: now also C12.1, J2.4 (Pin_4), J3.25 (Pin_25), J3.3 (Pin_3), J4.3 (Pin_3), R4.1, R6.2, SW2.2, U2.2 (VO)
- net BOOT0: now also R5.1, SW2.1
- net GND: now also C11.2, C12.2, C13.2, C14.2, C15.2, D1.2 (A), D2.1 (K), D3.1 (K), J1.A1 (GND), J1.A12 (GND), J1.B1 (GND), J1.B12 (GND), J1.S1 (SHIELD), J2.1 (Pin_1), J3.1 (Pin_1), J4.1 (Pin_1), J4.25 (Pin_25), R1.1, R2.1, R5.2, SW1.2, U2.1 (GND), U3.2 (GND), Y1.2 (G), Y1.4 (G)
- net NRST: now also C15.1, R4.2, SW1.1
- net PC2: now reaches U1.10 (PC2)
- net PC2: now also J4.20 (Pin_20)
- net PC3: now reaches U1.11 (PC3)
- net PC3: now also J4.21 (Pin_21)
- net PA0: now reaches U1.14 (PA0)
- net PA0: now also J4.22 (Pin_22)
- net PA1: now reaches U1.15 (PA1)
- net PA1: now also J4.23 (Pin_23)
- net PA2: now reaches U1.16 (PA2)
- net PA2: now also J4.24 (Pin_24)
- net PA3: now reaches U1.17 (PA3)
- net PA3: now also J3.24 (Pin_24)
- net PC13: now reaches U1.2 (PC13)
- net PC13: now also J4.15 (Pin_15)
- net PA4: now reaches U1.20 (PA4)
- net PA4: now also J3.23 (Pin_23)
- net PA5: now reaches U1.21 (PA5)
- net PA5: now also J3.22 (Pin_22)
- net PA6: now reaches U1.22 (PA6)
- net PA6: now also J3.21 (Pin_21)
- net PA7: now reaches U1.23 (PA7)
- net PA7: now also J3.20 (Pin_20)
- net PC4: now reaches U1.24 (PC4)
- net PC4: now also J3.19 (Pin_19)
- net PC5: now reaches U1.25 (PC5)
- net PC5: now also J3.18 (Pin_18)
- net PB0: now reaches U1.26 (PB0)
- net PB0: now also J3.17 (Pin_17)
- net PB1: now reaches U1.27 (PB1)
- net PB1: now also J3.16 (Pin_16)
- net PB2: now reaches U1.28 (PB2)
- net PB2: now also J3.15 (Pin_15)
- net PB10: now reaches U1.29 (PB10)
- net PB10: now also J3.14 (Pin_14)
- net PC14: now reaches U1.3 (PC14)
- net PC14: now also J4.16 (Pin_16)
- net PB12: now reaches U1.33 (PB12)
- net PB12: now also J3.13 (Pin_13)
- net PB13: now reaches U1.34 (PB13)
- net PB13: now also J3.12 (Pin_12)
- net PB14: now reaches U1.35 (PB14)
- net PB14: now also J3.11 (Pin_11)
- net PB15: now reaches U1.36 (PB15)
- net PB15: now also J3.10 (Pin_10)
- net PC6: now reaches U1.37 (PC6)
- net PC6: now also J3.9 (Pin_9)
- net PC7: now reaches U1.38 (PC7)
- net PC7: now also J3.8 (Pin_8)
- net PC9: now reaches U1.39 (PC9)
- net PC9: now also J3.7 (Pin_7)
- net PC15: now reaches U1.4 (PC15)
- net PC15: now also J4.17 (Pin_17)
- net PA8: now reaches U1.40 (PA8)
- net PA8: now also J3.6 (Pin_6)
- net PA9: now reaches U1.41 (PA9)
- net PA9: now also J3.5 (Pin_5)
- net PA10: now reaches U1.42 (PA10)
- net PA10: now also J3.4 (Pin_4)
- net USB_D-: now reaches U1.43 (PA11)
- net USB_D-: now also U3.3 (I/O2)
- net USB_D+: now reaches U1.44 (PA12)
- net USB_D+: now also U3.1 (I/O1)
- net SWDIO: now reaches U1.45 (PA13)
- net SWDIO: now also J2.3 (Pin_3)
- net SWCLK: now reaches U1.49 (PA14)
- net SWCLK: now also J2.2 (Pin_2)
- net OSC_IN: now reaches U1.5 (PH0)
- net OSC_IN: now also C13.1, Y1.1
- net PA15: now reaches U1.50 (PA15)
- net PA15: now also J4.4 (Pin_4), R3.2
- net PC10: now reaches U1.51 (PC10)
- net PC10: now also J4.5 (Pin_5)
- net PC11: now reaches U1.52 (PC11)
- net PC11: now also J4.6 (Pin_6)
- net PC12: now reaches U1.53 (PC12)
- net PC12: now also J4.7 (Pin_7)
- net PD2: now reaches U1.54 (PD2)
- net PD2: now also J4.8 (Pin_8)
- net PB3: now reaches U1.55 (PB3)
- net PB3: now also J4.9 (Pin_9)
- net PB4: now reaches U1.56 (PB4)
- net PB4: now also J4.10 (Pin_10)
- net PB5: now reaches U1.57 (PB5)
- net PB5: now also J4.11 (Pin_11)
- net PB6: now reaches U1.58 (PB6)
- net PB6: now also J4.12 (Pin_12)
- net PB7: now reaches U1.59 (PB7)
- net PB7: now also J4.13 (Pin_13)
- net OSC_OUT: now reaches U1.6 (PH1)
- net OSC_OUT: now also C14.1, Y1.3
- net PB8: now reaches U1.61 (PB8)
- net PB8: now also J4.14 (Pin_14)
- net PB9: now reaches U1.62 (PB9)
- net PC0: now reaches U1.8 (PC0)
- net PC0: now also J4.18 (Pin_18)
- net PC1: now reaches U1.9 (PC1)
- net PC1: now also J4.19 (Pin_19)
- new net: D2.2 (A), R3.1
- new net: D3.2 (A), R6.1
- new net CC1: J1.A5 (CC1), R1.2
- new net CC2: J1.B5 (CC2), R2.2
- new net USB_CONN_D+: J1.A6 (D+), J1.B6 (D+), U3.6 (I/O1)
- new net USB_CONN_D-: J1.A7 (D-), J1.B7 (D-), U3.4 (I/O2)
- new net VBUS: C11.1, D1.1 (K), J1.A4 (VBUS), J1.A9 (VBUS), J1.B4 (VBUS), J1.B9 (VBUS), J3.2 (Pin_2), J4.2 (Pin_2), U2.3 (VI), U3.5 (VBUS)
Other:
- note added: "BOOTSEL Button"
- note added: "BOOTSEL allows USB DFU programming when pulled high during reset"
- note added: "BOOTSEL boots and runs from flash when pulled low"
- note added: "C = (Lc / 2) - 2pF (-2pF for trace parasitic capacitance)"
- note added: "Capacitor acts like GND short on powerup, resetting the MCU"
- note added: "Crystal Oscillator"
- note added: "Crystal oscillator allows better timing than MCU internal RC clock"
- note added: "Linear Voltage Regulator"
- note added: "Load caps from crystal load capacitance"
- note added: "Pulldown resistor prevents floating BOOTSEL (inconsistent MCU boot behavior)"
- note added: "Pullup resistor prevents floating reset (unwanted resets of MCU)"
- note added: "RESET Button"
- note added: "RESET is active low"
- note added: "USB Connector & ESD Protection"
- moved on the sheet: C1, C10, C2, C3, C4, C5, C6, C7, C8, C9, U1

Commit message: QSPI DRAM support
Parts:
- removed J3, J4: Conn_01x25_PinHeader, Connector_PinHeader_2.54mm:PinHeader_1x25_P2.54mm_Vertical, symbol Connector:Conn_01x25_Socket
- added J3, J4: Conn_01x22_Socket, Connector_PinHeader_2.54mm:PinHeader_1x22_P2.54mm_Vertical, symbol Connector:Conn_01x22_Socket
- added U4: APS6404L-3SQR-SN, Package_SO:SOIC-8_3.9x4.9mm_P1.27mm, symbol Memory_RAM:APS6404L-3SQRx-SN
- C10, C2: footprint Capacitor_SMD:C_0402_1005Metric_Pad0.74x0.62mm_HandSolder -> Capacitor_SMD:C_0603_1608Metric
Connections:
- net +3V3: now also J3.22 (Pin_22), J3.3 (Pin_3), J4.3 (Pin_3), U4.8 (VDD)
- net GND: now also J3.1 (Pin_1), J4.1 (Pin_1), J4.22 (Pin_22), U4.4 (VSS)
- net PA0: now also J4.20 (Pin_20)
- net PA1: now also U4.7 (SIO3)
- net PA10: now also J3.4 (Pin_4)
- net PA15: now also J4.4 (Pin_4)
- net PA2: now also J4.21 (Pin_21)
- net PA3: now also U4.6 (SCLK)
- net PA4: now also J3.21 (Pin_21)
- net PA5: now also J3.20 (Pin_20)
- net PA6: now also J3.19 (Pin_19)
- net PA7: now also J3.18 (Pin_18)
- net PA8: now also J3.6 (Pin_6)
- net PA9: now also J3.5 (Pin_5)
- net PB0: now also U4.2 (SO/SIO1)
- net PB1: now also J3.15 (Pin_15)
- net PB10: now also U4.1 (~{CE})
- net PB12: now also J3.13 (Pin_13)
- net PB13: now also J3.12 (Pin_12)
- net PB14: now also J3.11 (Pin_11)
- net PB15: now also J3.10 (Pin_10)
- net PB2: now also J3.14 (Pin_14)
- net PB3: now also J4.9 (Pin_9)
- net PB4: now also J4.10 (Pin_10)
- net PB5: now also J4.11 (Pin_11)
- net PB6: now also J4.12 (Pin_12)
- net PB7: now also J4.13 (Pin_13)
- net PB8: now also J4.14 (Pin_14)
- net PC0: now also J4.18 (Pin_18)
- net PC1: now also J4.19 (Pin_19)
- net PC10: now also J4.5 (Pin_5)
- net PC11: now also J4.6 (Pin_6)
- net PC12: now also J4.7 (Pin_7)
- net PC13: now also J4.15 (Pin_15)
- net PC14: now also J4.16 (Pin_16)
- net PC15: now also J4.17 (Pin_17)
- net PC2: now also U4.3 (SIO2)
- net PC3: now also U4.5 (SI/SIO0)
- net PC4: now also J3.17 (Pin_17)
- net PC5: now also J3.16 (Pin_16)
- net PC6: now also J3.9 (Pin_9)
- net PC7: now also J3.8 (Pin_8)
- net PC9: now also J3.7 (Pin_7)
- net PD2: now also J4.8 (Pin_8)
- net VBUS: now also J3.2 (Pin_2), J4.2 (Pin_2)
